File: extended/pcb/pcb.kicad_pcb (KiCad board)
At the start: 2 copper layers, 100 x 84.5 mm, 27 parts, among them J1 LED Out +24V, J2 LED Out data, J3 LED Out GND, J4 5V out, J5 Power in 24V, J6 MEZD71201A-G, J7 Power in GND, K1 AZ943-1CH-5DE, U1 WLED, U2 74HCT245

Commit message: fix relay flickering on boot
Connections:
- U1 pad 14: unconnected-(U1-SCL/D1-Pad14) -> Net-(U1-SCL/D1)
- U1 pad 6: Net-(U1-MOSI/D7) -> unconnected-(U1-MOSI/D7-Pad6)
- U2 pad 4: Net-(U1-MOSI/D7) -> Net-(U1-SCL/D1)
Routing:
- net Net-(U1-SCL/D1): track 0.00 -> 28.8 mm
- net Net-(U1-MOSI/D7): track 24.7 -> 0.00 mm
- net Net-(U1-TX): track 36.1 -> 33.9 mm
- net +5VD: track 98.2 -> 96.7 mm
- net Net-(U2-B2): vias 0 -> 1
Other:
- board text added: "Configure Relay with GPIO 5"
- board text removed: "Configure Relay with GPIO13"
Changed lines of the file:
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@@
 	(net 0 "")
 	(net 1 "GND")
-	(net 2 "Net-(J9-Pin_1)")
-	(net 3 "Net-(J9-Pin_3)")
+	(net 2 "Net-(J6-Pin_1)")
+	(net 3 "Net-(J6-Pin_3)")
 	(net 4 "+5VD")
 	(net 5 "Net-(D1-A)")
-	(net 6 "Net-(J4-Pin_2)")
-	(net 7 "Net-(J4-Pin_1)")
+	(net 6 "Net-(J1-Pin_2)")
+	(net 7 "Net-(J1-Pin_1)")
 	(net 8 "+24V")
-	(net 9 "Net-(J7-Pin_1)")
-	(net 10 "Net-(J7-Pin_2)")
+	(net 9 "Net-(J2-Pin_1)")
+	(net 10 "Net-(J2-Pin_2)")
 	(net 11 "unconnected-(K1-Pad4)")
 	(net 12 "Net-(U2-B2)")
@@
 	(net 19 "unconnected-(U1-~{RST}-Pad1)")
 	(net 20 "unconnected-(U1-D0-Pad3)")
-	(net 21 "Net-(U1-MOSI{slash}D7)")
+	(net 21 "unconnected-(U1-MOSI{slash}D7-Pad6)")
 	(net 22 "unconnected-(U1-D3-Pad12)")
 	(net 23 "unconnected-(U1-RX-Pad15)")
@@
 	(net 25 "unconnected-(U1-CS{slash}D8-Pad7)")
 	(net 26 "unconnected-(U1-A0-Pad2)")
-	(net 27 "unconnected-(U1-SCL{slash}D1-Pad14)")
+	(net 27 "Net-(U1-SCL{slash}D1)")
 	(net 28 "Net-(U1-D4)")
 	(net 29 "unconnected-(U2-B4-Pad14)")
@@
 			(layers "*.Cu" "*.Mask")
 			(remove_unused_layers no)
-			(net 7 "Net-(J4-Pin_1)")
+			(net 7 "Net-(J1-Pin_1)")
 			(pinfunction "Pin_1")
 			(pintype "power_out")
@@
 			(layers "*.Cu" "*.Mask")
 			(remove_unused_layers no)
-			(net 6 "Net-(J4-Pin_2)")
+			(net 6 "Net-(J1-Pin_2)")
 			(pinfunction "Pin_2")
 			(pintype "power_out")
@@
 			(layers "*.Cu" "*.Mask")
 			(remove_unused_layers no)
-			(net 3 "Net-(J9-Pin_3)")
+			(net 3 "Net-(J6-Pin_3)")
 			(pintype "passive")
 		)
@@
 			(layers "*.Cu" "*.Mask")
 			(remove_unused_layers no)
-			(net 7 "Net-(J4-Pin_1)")
+			(net 7 "Net-(J1-Pin_1)")
 			(pinfunction "3")
 			(pintype "unspecified")
@@
 			(layers "*.Cu" "*.Mask")
 			(remove_unused_layers no)
-			(net 7 "Net-(J4-Pin_1)")
+			(net 7 "Net-(J1-Pin_1)")
 			(pinfunction "4")
 			(pintype "unspecified")
@@
 			(layers "*.Cu" "*.Mask")
 			(remove_unused_layers no)
-			(net 10 "Net-(J7-Pin_2)")
+			(net 10 "Net-(J2-Pin_2)")
 			(pintype "passive")
 		)
@@
 			(layers "*.Cu" "*.Mask")
 			(remove_unused_layers no)
-			(net 2 "Net-(J9-Pin_1)")
+			(net 2 "Net-(J6-Pin_1)")
 			(pintype "passive")
 		)
@@
 			(layers "*.Cu" "*.Mask")
 			(remove_unused_layers no)
-			(net 2 "Net-(J9-Pin_1)")
+			(net 2 "Net-(J6-Pin_1)")
 			(pintype "passive")
 		)
@@
 			(layers "*.Cu" "*.Mask")
 			(remove_unused_layers no)
-			(net 9 "Net-(J7-Pin_1)")
+			(net 9 "Net-(J2-Pin_1)")
 			(pintype "passive")
 		)
@@
 			(layers "*.Cu" "*.Mask")
 			(remove_unused_layers no)
-			(net 21 "Net-(U1-MOSI{slash}D7)")
+			(net 27 "Net-(U1-SCL{slash}D1)")
 			(pinfunction "A2")
 			(pintype "tri_state")
@@
 		(tags "Through hole socket strip THT 1x03 2.54mm single row")
 		(property "Reference" "J6"
-			(at 0 -2.77 360)
+			(at 0 -2.77 0)
 			(layer "F.SilkS")
 			(effects
@@
 		)
 		(property "Value" "MEZD71201A-G"
-			(at 0 7.85 360)
+			(at 0 7.85 0)
 			(layer "F.Fab")
 			(effects
@@
 			(layers "*.Cu" "*.Mask")
 			(remove_unused_layers no)
-			(net 2 "Net-(J9-Pin_1)")
+			(net 2 "Net-(J6-Pin_1)")
 			(pinfunction "Pin_1")
 			(pintype "passive")
@@
 			(layers "*.Cu" "*.Mask")
 			(remove_unused_layers no)
-			(net 3 "Net-(J9-Pin_3)")
+			(net 3 "Net-(J6-Pin_3)")
 			(pinfunction "Pin_3")
 			(pintype "passive")
@@
 			(layers "*.Cu" "*.Mask")
 			(remove_unused_layers no)
-			(net 21 "Net-(U1-MOSI{slash}D7)")
+			(net 21 "unconnected-(U1-MOSI{slash}D7-Pad6)")
 			(pinfunction "MOSI/D7")
-			(pintype "bidirectional")
+			(pintype "bidirectional+no_connect")
 		)
 		(pad "7" thru_hole oval
@@
 			(layers "*.Cu" "*.Mask")
 			(remove_unused_layers no)
-			(net 27 "unconnected-(U1-SCL{slash}D1-Pad14)")
+			(net 27 "Net-(U1-SCL{slash}D1)")
 			(pinfunction "SCL/D1")
-			(pintype "bidirectional+no_connect")
+			(pintype "bidirectional")
 		)
 		(pad "15" thru_hole oval
@@
 			(layers "*.Cu" "*.Mask")
 			(remove_unused_layers no)
-			(net 3 "Net-(J9-Pin_3)")
+			(net 3 "Net-(J6-Pin_3)")
 			(pintype "passive")
 		)
@@
 			(layers "*.Cu" "*.Mask")
 			(remove_unused_layers no)
-			(net 6 "Net-(J4-Pin_2)")
+			(net 6 "Net-(J1-Pin_2)")
 			(pinfunction "3")
 			(pintype "unspecified")
@@
 			(layers "*.Cu" "*.Mask")
 			(remove_unused_layers no)
-			(net 6 "Net-(J4-Pin_2)")
+			(net 6 "Net-(J1-Pin_2)")
 			(pinfunction "4")
 			(pintype "unspecified")
@@
 			(layers "*.Cu" "*.Mask")
 			(remove_unused_layers no)
-			(net 9 "Net-(J7-Pin_1)")
+			(net 9 "Net-(J2-Pin_1)")
 			(pinfunction "Pin_1")
 			(pintype "passive")
@@
 			(layers "*.Cu" "*.Mask")
 			(remove_unused_layers no)
-			(net 10 "Net-(J7-Pin_2)")
+			(net 10 "Net-(J2-Pin_2)")
 			(pinfunction "Pin_2")
 			(pintype "passive")
@@
 		(tags "CP Radial series Radial pin pitch 2.00mm  diameter 5mm Electrolytic Capacitor")
 		(property "Reference" "C3"
-			(at 1 -3.75 360)
+			(at 1 -3.75 0)
 			(layer "F.SilkS")
 			(effects
@@
 		)
 		(property "Value" "C 10uF 5V optional (nah an level shifter)"
-			(at 1 3.75 360)
+			(at 1 3.75 0)
 			(layer "F.Fab")
 			(effects
@@
 		)
 		(fp_text user "${REFERENCE}"
-			(at 1 0 360)
+			(at 1 0 0)
 			(layer "F.Fab")
 			(effects
@@
 		)
 	)
-	(gr_text "Configure Relay with GPIO13"
+	(gr_text "Configure Relay with GPIO 5"
 		(at 183 74.5 0)
 		(layer "F.SilkS")
@@
 	(segment
 		(start 213 70)
-		(end 214.5 70)
-		(width 0.2)
-		(layer "F.Cu")
-		(net 4)
-	)
-	(segment
-		(start 213 70)
 		(end 202.489365 70)
 		(width 0.2)
@@
 	)
 	(segment
-		(start 153 95.5)
-		(end 157.88 90.62)
+		(start 157.88 90.62)
+		(end 153 95.5)
 		(width 0.2)
-		(layer "B.Cu")
+		(layer "F.Cu")
 		(net 12)
 	)
 	(segment
-		(start 147.76 95.5)
-		(end 153 95.5)
+		(start 170.88 90.62)
+		(end 157.88 90.62)
 		(width 0.2)
-		(layer "B.Cu")
+		(layer "F.Cu")
 		(net 12)
 	)
 	(segment
-		(start 140.455 102.805)
+		(start 153 95.5)
 		(end 147.76 95.5)
 		(width 0.2)
-		(layer "B.Cu")
+		(layer "F.Cu")
+		(net 12)
+	)
+	(via
+		(at 147.76 95.5)
+		(size 0.6)
+		(drill 0.3)
+		(layers "F.Cu" "B.Cu")
 		(net 12)
 	)
 	(segment
-		(start 157.88 90.62)
-		(end 170.88 90.62)
+		(start 140.455 102.805)
+		(end 147.76 95.5)
 		(width 0.2)
 		(layer "B.Cu")
@@
 	)
 	(segment
-		(start 178.5 98.24)
-		(end 179.76 98.24)
+		(start 183.26 103)
+		(end 206.805 103)
 		(width 0.2)
 		(layer "B.Cu")
@@
 	)
 	(segment
-		(start 209.39 96.89)
-		(end 209.39 100.415)
+		(start 178.5 98.24)
+		(end 183.26 103)
 		(width 0.2)
 		(layer "B.Cu")
@@
 	)
 	(segment
-		(start 179.76 98.24)
-		(end 182.5 95.5)
+		(start 206.805 103)
+		(end 209.39 100.415)
 		(width 0.2)
 		(layer "B.Cu")
@@
 	)
 	(segment
-		(start 208 95.5)
-		(end 209.39 96.89)
+		(start 178.5 93.16)
+		(end 197.055 93.16)
 		(width 0.2)
 		(layer "B.Cu")
-		(net 16)
+		(net 27)
 	)
 	(segment
-		(start 182.5 95.5)
-		(end 208 95.5)
+		(start 197.055 93.16)
+		(end 204.31 100.415)
 		(width 0.2)
 		(layer "B.Cu")
-		(net 16)
-	)
-	(segment
-		(start 196.69 77.555)
-		(end 181.085 93.16)
-		(width 0.2)
-		(layer "F.Cu")
-		(net 21)
-	)
-	(segment
-		(start 181.085 93.16)
-		(end 178.5 93.16)
-		(width 0.2)
-		(layer "F.Cu")
-		(net 21)
+		(net 27)
 	)
 	(segment

Commit message: This commit is most probably wrong, but lets store it
The issue is that when the PCB is provided power then the led strip
quickly lights up, then goes of. Afterwards wled turns it on again.

I though this is because the wiring of the relay is wrong. The
documentation shows the default state to be in reverse of what the
downloadbale schematic provides
(https://www.azettler.com/pdfs/az943.pdf).
Then the relay would be on when no power is applied through the coil.

However that does not really match the sounds it makes. During the quick
on time of the led strip there are two click sounds instead of one which
should be the case if the above holds true.
Unless the relay per default clicks once when power is provided even
when the coil is low.
Connections:
- K1 pad 2: Net-(U2-B2) -> GND
- K1 pad 3: +24V after Relay -> unconnected-(K1-Pad3)
- K1 pad 4: unconnected-(K1-Pad4) -> +24V after Relay
- K1 pad 5: GND -> Net-(U2-B2)
Routing:
- net Net-(U2-B2): track 35.5 -> 47.5 mm
- net GND: track 31.1 -> 19.8 mm
