File: extended/pcb/pcb.kicad_pcb (KiCad board)
At the start: 2 copper layers, 100 x 84.5 mm, 27 parts, among them J1 LED Out +24V, J2 LED Out data, J3 LED Out GND, J4 5V out, J5 Power in 24V, J6 MEZD71201A-G, J7 Power in GND, K1 AZ943-1CH-5DE, U1 WLED, U2 74HCT245

Commit message: add missing pulldown resistor
D1 does not have a pulldown resistor included, so the output is floating
during boot. This can cause the led strip to flicker.
Fix this by adding a pulldown resistor.
Parts:
- added R4: R 5.1k, Resistor_THT:R_Axial_DIN0207_L6.3mm_D2.5mm_P10.16mm_Horizontal, F.Cu at (195.5, 93.2)
Routing:
- net Net-(U1-D4): track 23.7 -> 20.1 mm
