File: extended/pcb/pcb.kicad_sch (KiCad schematic)
At the start: 23 parts, among them J1 LED Out +24V, J2 LED Out data, J3 LED Out GND, J4 5V out, J5 Power in 24V, J6 MEZD71201A-G, J7 Power in GND, K1 AZ943-1CH-5DE, U1 WLED, U2 74HCT245

Commit message: add missing pulldown resistor
D1 does not have a pulldown resistor included, so the output is floating
during boot. This can cause the led strip to flicker.
Fix this by adding a pulldown resistor.
Parts:
- added R4: R 5.1k, Resistor_THT:R_Axial_DIN0207_L6.3mm_D2.5mm_P10.16mm_Horizontal, symbol Device:R
Connections:
- net GND: now also R4.2
- net at U1.14 (SCL/D1), U2.4 (A2): now also R4.1
Changed lines of the file:
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@@
+	)
+	(junction
+		(at 129.54 119.38)
+		(diameter 0)
+		(color 0 0 0 0)
 	)
 	(junction
@@
 	)
 	(junction
+		(at 129.54 88.9)
+		(diameter 0)
+		(color 0 0 0 0)
+	)
+	(junction
 		(at 119.38 55.88)
 		(diameter 0)
@@
 	(wire
 		(pts
-			(xy 124.46 119.38) (xy 140.97 119.38)
+			(xy 124.46 119.38) (xy 129.54 119.38)
 		)
 		(stroke
@@
 	(wire
 		(pts
-			(xy 120.65 88.9) (xy 140.97 88.9)
+			(xy 120.65 88.9) (xy 129.54 88.9)
 		)
 		(stroke
@@
 	(wire
 		(pts
+			(xy 129.54 99.06) (xy 129.54 88.9)
+		)
+		(stroke
+			(width 0)
+			(type default)
+		)
+	)
+	(wire
+		(pts
 			(xy 50.8 53.34) (xy 50.8 116.84)
 		)
@@
 	(wire
 		(pts
+			(xy 129.54 106.68) (xy 129.54 119.38)
+		)
+		(stroke
+			(width 0)
+			(type default)
+		)
+	)
+	(wire
+		(pts
 			(xy 57.15 21.59) (xy 185.42 21.59)
 		)
@@
 	(wire
 		(pts
+			(xy 129.54 88.9) (xy 140.97 88.9)
+		)
+		(stroke
+			(width 0)
+			(type default)
+		)
+	)
+	(wire
+		(pts
 			(xy 226.06 68.58) (xy 226.06 119.38)
 		)
@@
 		(pts
 			(xy 124.46 119.38) (xy 124.46 121.92)
+		)
+		(stroke
+			(width 0)
+			(type default)
+		)
+	)
+	(wire
+		(pts
+			(xy 129.54 119.38) (xy 140.97 119.38)
 		)
 		(stroke
@@
 					(unit 1)
 				)
+			)
+		)
+	)
+	(symbol
+		(lib_id "Device:R")
+		(at 129.54 102.87 0)
+		(unit 1)
+		(exclude_from_sim no)
+		(in_bom yes)
+		(on_board yes)
+		(dnp no)
+		(property "Reference" "R4"
+			(at 124.46 101.6 0)
+			(effects
+				(font
+					(size 1.27 1.27)
+				)
+				(justify left)
+			)
+		)
+		(property "Value" "R 5.1k"
+			(at 121.666 104.394 0)
+			(effects
+				(font
+					(size 1.27 1.27)
+				)
+				(justify left)
+			)
+		)
+		(property "Footprint" "Resistor_THT:R_Axial_DIN0207_L6.3mm_D2.5mm_P10.16mm_Horizontal"
+			(at 127.762 102.87 90)
+			(effects
+				(font
+					(size 1.27 1.27)
+				)
+				(hide yes)
+			)
+		)
+		(property "Datasheet" "~"
+			(at 129.54 102.87 0)
+			(effects
+				(font
+					(size 1.27 1.27)
+				)
+				(hide yes)
+			)
+		)
+		(property "Description" "Resistor"
+			(at 129.54 102.87 0)
+			(effects
+				(font
+					(size 1.27 1.27)
+				)
+				(hide yes)
+			)
+		)
+		(pin "1"
+		)
+		(pin "2"
+		)
+		(instances
+			(project "pcb"
+				(path "/f9e27db9-af07-4f92-8184-1b5de79e3cda"
+					(reference "R4")
+					(unit 1)
+				)
